Commit message: fixes, docs, more complex example

File: gz_camera_macros/urdf/rgb_camera.gazebo.xacro (robot description, xacro)
@@ -53,9 +53,12 @@
                 <stddev>0.00</stddev>
               </noise>
+              <!-- TODO this term is deprecated but behaves better than setting
+                  '<gz_frame_id>${name}_color_optical_frame</gz_frame_id>'
+                  in the <sensor> namespace -->
               <optical_frame_id>${name}_color_optical_frame</optical_frame_id>
               <triggered>${triggered}</triggered>
               <trigger_topic>${name}/trigger</trigger_topic>
           </camera>
-          <gz_frame_id>${name}_color_frame</gz_frame_id>
+          <!-- <gz_frame_id>${name}_color_optical_frame</gz_frame_id> -->
           <always_on>1</always_on>
           <update_rate>${fps}</update_rate>
@@ -63,22 +66,4 @@
           <enable_metrics>false</enable_metrics>
         </sensor>
-        <sensor name="${name}_depth" type="depth">
-          <camera>
-            <horizontal_fov>${h_fov}</horizontal_fov>
-            <image>
-              <width>${image_width}</width>
-              <height>${image_height}</height>
-            </image>
-            <clip>
-              <near>0.1</near>
-              <far>10</far>
-            </clip>
-          </camera>
-          <gz_frame_id>${name}_color_frame</gz_frame_id>
-          <always_on>1</always_on>
-          <update_rate>${fps}</update_rate>
-          <topic>${gz_topic_name}/depth_image</topic>
-          <enable_metrics>false</enable_metrics>
-        </sensor>
     </gazebo>
 </xacro:macro>

File: gz_camera_macros/urdf/rgbd_camera.gazebo.xacro (robot description, xacro)
@@ -84,4 +84,7 @@
                     </clip>
                 </depth_camera>
+                <!-- TODO this term is deprecated but behaves better than setting
+                    '<gz_frame_id>${name}_color_optical_frame</gz_frame_id>'
+                    in the <sensor> namespace -->
                 <optical_frame_id>${name}_color_optical_frame</optical_frame_id>
             </camera>

File: orbbec_gz_description/urdf/example_335Le_gazebo.urdf.xacro (robot description, xacro)
@@ -22,4 +22,4 @@
   </gazebo>
   <!-- The xacros included in this repo assume the same link/joint names as gemini335Le when passed the same name -->
-  <xacro:gazebo_gemini335Le name="$(arg camera_name)"/>
+  <xacro:gazebo_gemini335Le name="$(arg camera_name)" gz_topic_name="$(arg camera_name)" type="rgb+d"/>
 </robot>

File: orbbec_gz_description/urdf/gemini335Le.gazebo.xacro (robot description, xacro)
@@ -2,4 +2,5 @@
 <robot name="gazebo_gemini335Le" xmlns:xacro="http://www.ros.org/wiki/xacro" xmlns:gz="http://gazebosim.org/schema">
 <xacro:include filename="$(find gz_camera_macros)/urdf/rgb_camera.gazebo.xacro" />
+<xacro:include filename="$(find gz_camera_macros)/urdf/depth_camera.gazebo.xacro" />
 <xacro:include filename="$(find gz_camera_macros)/urdf/rgbd_camera.gazebo.xacro" />
 <!-- Xacro args
@@ -33,4 +34,11 @@
     <xacro:property name="min_depth" value="0.25" />
     <xacro:property name="max_depth" value="6.0" />
+    <!--
+    For this camera to work correctly we need to have a joint to attach to and Gazebo collapses fixed joints by default.
+    This preserves the camera_color_joint so that the camera_color_frame where the sensor is located is available.
+    -->
+    <gazebo reference='${name}_color_joint'>
+      <disableFixedJointLumping>true</disableFixedJointLumping>
+    </gazebo>
     <xacro:if value="${type == 'rgbd'}">
         <xacro:gazebo_rgbd name="${name}"
@@ -54,4 +62,22 @@
                         triggered="${triggered}"/>
     </xacro:if>
+    <xacro:if value="${type == 'rgb+d'}">
+        <xacro:gazebo_rgb name="${name}"
+                          fps="${fps}"
+                          gz_topic_name="${gz_topic_name}"
+                          image_width="${image_width}"
+                          image_height="${image_height}"
+                          h_fov="${realsense_h_fov}"
+                          v_fov="${realsense_v_fov}"
+                          triggered="${triggered}"/>
+        <xacro:gazebo_depth name="${name}"
+                            fps="${fps}"
+                            gz_topic_name="${gz_topic_name}"
+                            image_width="${image_width}"
+                            image_height="${image_height}"
+                            h_fov="${realsense_h_fov}"
+                            v_fov="${realsense_v_fov}"
+                            triggered="${triggered}"/>
+    </xacro:if>
 </xacro:macro>
 </robot>

File: realsense2_gz_description/urdf/_d415.gazebo.xacro (robot description, xacro)
@@ -2,4 +2,5 @@
 <robot name="gazebo_d415" xmlns:xacro="http://www.ros.org/wiki/xacro" xmlns:gz="http://gazebosim.org/schema">
 <xacro:include filename="$(find gz_camera_macros)/urdf/rgb_camera.gazebo.xacro" />
+<xacro:include filename="$(find gz_camera_macros)/urdf/depth_camera.gazebo.xacro" />
 <xacro:include filename="$(find gz_camera_macros)/urdf/rgbd_camera.gazebo.xacro" />
 <!-- Xacro args
@@ -33,4 +34,7 @@
     <xacro:property name="min_depth" value="0.45" />
     <xacro:property name="max_depth" value="3.0" />
+    <!-- <gazebo reference='${name}_color_joint'>
+      <disableFixedJointLumping>true</disableFixedJointLumping>
+    </gazebo>  -->
     <xacro:if value="${type == 'rgbd'}">
         <xacro:gazebo_rgbd name="${name}"
@@ -46,11 +50,29 @@
     <xacro:if value="${type == 'rgb'}">
         <xacro:gazebo_rgb name="${name}"
-                        fps="${fps}"
-                        gz_topic_name="${gz_topic_name}"
-                        image_width="${image_width}"
-                        image_height="${image_height}"
-                        h_fov="${realsense_h_fov}"
-                        v_fov="${realsense_v_fov}"
-                        triggered="${triggered}"/>
+                          fps="${fps}"
+                          gz_topic_name="${gz_topic_name}"
+                          image_width="${image_width}"
+                          image_height="${image_height}"
+                          h_fov="${realsense_h_fov}"
+                          v_fov="${realsense_v_fov}"
+                          triggered="${triggered}"/>
+    </xacro:if>
+    <xacro:if value="${type == 'rgb+d'}">
+        <xacro:gazebo_rgb name="${name}"
+                          fps="${fps}"
+                          gz_topic_name="${gz_topic_name}"
+                          image_width="${image_width}"
+                          image_height="${image_height}"
+                          h_fov="${realsense_h_fov}"
+                          v_fov="${realsense_v_fov}"
+                          triggered="${triggered}"/>
+        <xacro:gazebo_depth name="${name}"
+                            fps="${fps}"
+                            gz_topic_name="${gz_topic_name}"
+                            image_width="${image_width}"
+                            image_height="${image_height}"
+                            h_fov="${realsense_h_fov}"
+                            v_fov="${realsense_v_fov}"
+                            triggered="${triggered}"/>
     </xacro:if>
 </xacro:macro>

File: realsense2_gz_description/urdf/example_d415_gazebo.urdf.xacro (robot description, xacro)
@@ -1,5 +1,4 @@
 <?xml version="1.0"?>
 <robot name="realsense2_gz_camera" xmlns:xacro="http://ros.org/wiki/xacro">
-  <xacro:arg name="camera_name" default="camera" />
   <xacro:arg name="add_plug" default="false" />
   <xacro:arg name="use_mesh" default="true" />
@@ -11,12 +10,25 @@
   <link name="world" /> <!-- The parent of the camera in this example is the Gazebo world -->
   <!-- Call the URDF xacro. -->
-  <xacro:sensor_d415 parent="world" name="$(arg camera_name)" use_nominal_extrinsics="${use_nominal_extrinsics}" add_plug="$(arg add_plug)" use_mesh="$(arg use_mesh)">
+  <xacro:sensor_d415 parent="world" name="forward_camera" use_nominal_extrinsics="${use_nominal_extrinsics}" add_plug="$(arg add_plug)" use_mesh="$(arg use_mesh)">
     <!-- Place the camera above the ground and point it down a little to look at the objects in the scene -->
     <origin xyz="0 0 0.5" rpy="0 0.1 0"/>
   </xacro:sensor_d415>
+  <!-- The xacros included in this repo assume the same link/joint names as sensor_d415 when passed the same name -->
+  <xacro:gazebo_d415 name="forward_camera" gz_topic_name="forward_camera" type="rgb+d" fps="5"/>
+  <!-- Camera on the left -->
+  <xacro:sensor_d415 parent="world" name="left_camera" use_nominal_extrinsics="${use_nominal_extrinsics}" add_plug="$(arg add_plug)" use_mesh="$(arg use_mesh)">
+    <origin xyz="1.2 1.5 0.5" rpy="0 0.1 ${-pi/2}"/>
+  </xacro:sensor_d415>
+  <xacro:gazebo_d415 name="left_camera" gz_topic_name="left_camera" type="rgb+d" fps="5"/>
+  <!-- Canera on the right -->
+  <xacro:sensor_d415 parent="world" name="right_camera" use_nominal_extrinsics="${use_nominal_extrinsics}" add_plug="$(arg add_plug)" use_mesh="$(arg use_mesh)">
+    <origin xyz="1.2 -1.5 0.5" rpy="0 0.1 ${pi/2}"/>
+  </xacro:sensor_d415>
+  <xacro:gazebo_d415 name="right_camera" gz_topic_name="right_camera" type="rgb+d" fps="5"/>
   <!--
   This example xacro is the top parent so we need to include the Gazebo Sensor plugin here so the camera we define in the xarco below works.
   Starting this plugin in the top level allows developers to define multiple cameras in their robot and only include the plugin once.
-  If you don't want to start the Sensors plugin in your URDF you can move starting this plugin to the world.sdf file you are working with. -->
+  If you don't want to start the Sensors plugin in your URDF you can move starting this plugin to the world.sdf file you are working with.
+  -->
   <gazebo>
     <plugin filename="gz-sim-sensors-system" name="gz::sim::systems::Sensors">
@@ -24,5 +36,3 @@
     </plugin>
   </gazebo>
-  <!-- The xacros included in this repo assume the same link/joint names as sensor_d415 when passed the same name -->
-  <xacro:gazebo_d415 name="$(arg camera_name)"/>
 </robot>
