Commit message: General gz camera (#5)

File: gz_camera_macros/urdf/rgbd_camera.gazebo.xacro (robot description, xacro)
@@ -84,4 +84,7 @@
                     </clip>
                 </depth_camera>
+                <!-- WARNING
+                    This term is deprecated and the point clouds published from this sensor have the incorrect frame_id associated with the data.
+                -->
                 <optical_frame_id>${name}_color_optical_frame</optical_frame_id>
             </camera>

File: orbbec_gz_description/urdf/gemini335L_336Lgazebo.xacro (robot description, xacro)
@@ -1,18 +1,18 @@
 <?xml version="1.0"?>
-<robot name="gazebo_d435" xmlns:xacro="http://www.ros.org/wiki/xacro" xmlns:gz="http://gazebosim.org/schema">
-<xacro:include filename="$(find realsense2_gz_description)/urdf/rgb_camera.gazebo.xacro" />
-<xacro:include filename="$(find realsense2_gz_description)/urdf/rgbd_camera.gazebo.xacro" />
+<robot name="gazebo_gemini_335L_336L" xmlns:xacro="http://www.ros.org/wiki/xacro" xmlns:gz="http://gazebosim.org/schema">
+<xacro:include filename="$(find gz_camera_macros)/urdf/rgb_camera.gazebo.xacro" />
+<xacro:include filename="$(find gz_camera_macros)/urdf/rgbd_camera.gazebo.xacro" />
 <!-- Xacro args
-    name: should match the name value passed to realsense2_description sensor xacro
+    name: should match the name value passed to orbbec_description sensor xacro
     type:  valid values [rgb or rgbd]. Sensor type you would like to simulate
     fps: the target frame rate of the camera images
     gz_topic_name: the topic name the image and camera_info are published to Gazebo topics
-    image_width: See Realsense documentation for what the physical sensor supports
-    image_height: See Realsense documentation for what the physical sensor supports
+    image_width: See Orbbec documentation for what the physical sensor supports
+    image_height: See Orbbec documentation for what the physical sensor supports
     trigger: valid values [true, false]. Only supported with 'type=rgb' and will only publish a single image when triggered on Gazebo topic '${name}/trigger'
              example command line trigger
              ign topic -t "/name/trigger" -m Boolean -p "data: true" -n 1
 -->
-<xacro:macro name="gazebo_d435" params="
+<xacro:macro name="gazebo_gemini_335L_336L" params="
   name:=camera
   type:=rgbd
@@ -22,5 +22,5 @@
   image_height:=720
   triggered:=false">
-    <!-- Realsense D435 RGB properties
+    <!-- Orbbec gemini_335L_336L RGB properties
     Assumptions:
     Parent system (URDF or sdf) will start the Gazebo Sensors plugin. See notes in the camera.gazebo.xacros.
@@ -29,8 +29,10 @@
     Note: physical hardware publishes pointcloud in `camera_depth_optical_frame` where this sensor will use
     the referenced camera color_frame. -->
-    <xacro:property name="realsense_h_fov" value="${69 * pi/180}" />
-    <xacro:property name="realsense_v_fov" value="${42 * pi/180}" />
-    <xacro:property name="min_depth" value="0.28" />
-    <xacro:property name="max_depth" value="3.0" />
+    <!-- note that the depth FOV is slightly different, 90-deg x 65-deg.
+    https://store.orbbec.com/products/gemini-335l -->
+    <xacro:property name="realsense_h_fov" value="${94 * pi/180}" />
+    <xacro:property name="realsense_v_fov" value="${68 * pi/180}" />
+    <xacro:property name="min_depth" value="0.17" />
+    <xacro:property name="max_depth" value="6.0" />
     <xacro:if value="${type == 'rgbd'}">
         <xacro:gazebo_rgbd name="${name}"

File: realsense2_gz_description/urdf/_d405.gazebo.xacro (robot description, xacro)
@@ -1,6 +1,6 @@
 <?xml version="1.0"?>
-<robot name="gazebo_d455" xmlns:xacro="http://www.ros.org/wiki/xacro" xmlns:gz="http://gazebosim.org/schema">
-<xacro:include filename="$(find realsense2_gz_description)/urdf/rgb_camera.gazebo.xacro" />
-<xacro:include filename="$(find realsense2_gz_description)/urdf/rgbd_camera.gazebo.xacro" />
+<robot name="gazebo_d405" xmlns:xacro="http://www.ros.org/wiki/xacro" xmlns:gz="http://gazebosim.org/schema">
+<xacro:include filename="$(find gz_camera_macros)/urdf/rgb_camera.gazebo.xacro" />
+<xacro:include filename="$(find gz_camera_macros)/urdf/rgbd_camera.gazebo.xacro" />
 <!-- Xacro args
     name: should match the name value passed to realsense2_description sensor xacro
@@ -14,5 +14,5 @@
              ign topic -t "/name/trigger" -m Boolean -p "data: true" -n 1
 -->
-<xacro:macro name="gazebo_d455" params="
+<xacro:macro name="gazebo_d405" params="
   name:=camera
   type:=rgbd
@@ -22,5 +22,5 @@
   image_height:=720
   triggered:=false">
-    <!-- Realsense D455 RGB properties
+    <!-- Realsense D405 RGB properties
     Assumptions:
     Parent system (URDF or sdf) will start the Gazebo Sensors plugin. See notes in the camera.gazebo.xacros.
@@ -29,8 +29,8 @@
     Note: physical hardware publishes pointcloud in `camera_depth_optical_frame` where this sensor will use
     the referenced camera color_frame. -->
-    <xacro:property name="realsense_h_fov" value="${90 * pi/180}" />
-    <xacro:property name="realsense_v_fov" value="${65 * pi/180}" />
-    <xacro:property name="min_depth" value="0.52" />
-    <xacro:property name="max_depth" value="6.0" />
+    <xacro:property name="realsense_h_fov" value="${87 * pi/180}" />
+    <xacro:property name="realsense_v_fov" value="${58 * pi/180}" />
+    <xacro:property name="min_depth" value="0.07" />
+    <xacro:property name="max_depth" value="0.5" />
     <xacro:if value="${type == 'rgbd'}">
         <xacro:gazebo_rgbd name="${name}"

File: realsense2_gz_description/urdf/_d415.gazebo.xacro (robot description, xacro)
@@ -1,6 +1,7 @@
 <?xml version="1.0"?>
 <robot name="gazebo_d415" xmlns:xacro="http://www.ros.org/wiki/xacro" xmlns:gz="http://gazebosim.org/schema">
-<xacro:include filename="$(find realsense2_gz_description)/urdf/rgb_camera.gazebo.xacro" />
-<xacro:include filename="$(find realsense2_gz_description)/urdf/rgbd_camera.gazebo.xacro" />
+<xacro:include filename="$(find gz_camera_macros)/urdf/rgb_camera.gazebo.xacro" />
+<xacro:include filename="$(find gz_camera_macros)/urdf/depth_camera.gazebo.xacro" />
+<xacro:include filename="$(find gz_camera_macros)/urdf/rgbd_camera.gazebo.xacro" />
 <!-- Xacro args
     name: should match the name value passed to realsense2_description sensor xacro
@@ -33,4 +34,7 @@
     <xacro:property name="min_depth" value="0.45" />
     <xacro:property name="max_depth" value="3.0" />
+    <!-- <gazebo reference='${name}_color_joint'>
+      <disableFixedJointLumping>true</disableFixedJointLumping>
+    </gazebo>  -->
     <xacro:if value="${type == 'rgbd'}">
         <xacro:gazebo_rgbd name="${name}"
@@ -46,11 +50,29 @@
     <xacro:if value="${type == 'rgb'}">
         <xacro:gazebo_rgb name="${name}"
-                        fps="${fps}"
-                        gz_topic_name="${gz_topic_name}"
-                        image_width="${image_width}"
-                        image_height="${image_height}"
-                        h_fov="${realsense_h_fov}"
-                        v_fov="${realsense_v_fov}"
-                        triggered="${triggered}"/>
+                          fps="${fps}"
+                          gz_topic_name="${gz_topic_name}"
+                          image_width="${image_width}"
+                          image_height="${image_height}"
+                          h_fov="${realsense_h_fov}"
+                          v_fov="${realsense_v_fov}"
+                          triggered="${triggered}"/>
+    </xacro:if>
+    <xacro:if value="${type == 'rgb+d'}">
+        <xacro:gazebo_rgb name="${name}"
+                          fps="${fps}"
+                          gz_topic_name="${gz_topic_name}"
+                          image_width="${image_width}"
+                          image_height="${image_height}"
+                          h_fov="${realsense_h_fov}"
+                          v_fov="${realsense_v_fov}"
+                          triggered="${triggered}"/>
+        <xacro:gazebo_depth name="${name}"
+                            fps="${fps}"
+                            gz_topic_name="${gz_topic_name}"
+                            image_width="${image_width}"
+                            image_height="${image_height}"
+                            h_fov="${realsense_h_fov}"
+                            v_fov="${realsense_v_fov}"
+                            triggered="${triggered}"/>
     </xacro:if>
 </xacro:macro>

File: realsense2_gz_description/urdf/_d455.gazebo.xacro (robot description, xacro)
@@ -1,6 +1,6 @@
 <?xml version="1.0"?>
-<robot name="gazebo_d405" xmlns:xacro="http://www.ros.org/wiki/xacro" xmlns:gz="http://gazebosim.org/schema">
-<xacro:include filename="$(find realsense2_gz_description)/urdf/rgb_camera.gazebo.xacro" />
-<xacro:include filename="$(find realsense2_gz_description)/urdf/rgbd_camera.gazebo.xacro" />
+<robot name="gazebo_d455" xmlns:xacro="http://www.ros.org/wiki/xacro" xmlns:gz="http://gazebosim.org/schema">
+<xacro:include filename="$(find gz_camera_macros)/urdf/rgb_camera.gazebo.xacro" />
+<xacro:include filename="$(find gz_camera_macros)/urdf/rgbd_camera.gazebo.xacro" />
 <!-- Xacro args
     name: should match the name value passed to realsense2_description sensor xacro
@@ -14,5 +14,5 @@
              ign topic -t "/name/trigger" -m Boolean -p "data: true" -n 1
 -->
-<xacro:macro name="gazebo_d405" params="
+<xacro:macro name="gazebo_d455" params="
   name:=camera
   type:=rgbd
@@ -22,5 +22,5 @@
   image_height:=720
   triggered:=false">
-    <!-- Realsense D405 RGB properties
+    <!-- Realsense D455 RGB properties
     Assumptions:
     Parent system (URDF or sdf) will start the Gazebo Sensors plugin. See notes in the camera.gazebo.xacros.
@@ -29,8 +29,8 @@
     Note: physical hardware publishes pointcloud in `camera_depth_optical_frame` where this sensor will use
     the referenced camera color_frame. -->
-    <xacro:property name="realsense_h_fov" value="${87 * pi/180}" />
-    <xacro:property name="realsense_v_fov" value="${58 * pi/180}" />
-    <xacro:property name="min_depth" value="0.07" />
-    <xacro:property name="max_depth" value="0.5" />
+    <xacro:property name="realsense_h_fov" value="${90 * pi/180}" />
+    <xacro:property name="realsense_v_fov" value="${65 * pi/180}" />
+    <xacro:property name="min_depth" value="0.52" />
+    <xacro:property name="max_depth" value="6.0" />
     <xacro:if value="${type == 'rgbd'}">
         <xacro:gazebo_rgbd name="${name}"
